Commit message: trying to make better mu1, mu2

File: ias0220_224772/urdf/differential_robot_simu_task4_part1.urdf (robot description, URDF)
Before this commit: robot IAS0220_Evgenia, 7 links, 6 joints
Joints:
- joint base_to_left_wheel: limit effort=30 velocity=1.0 -> (none)
- joint base_to_right_wheel: limit effort=30 velocity=1.0 -> (none)

Commit message: add changes

File: ias0220_224772/urdf/differential_robot_simu_task4_part1.urdf (robot description, URDF)
Before this commit: robot IAS0220_Evgenia, 7 links, 6 joints
Joints:
- joint base_to_left_wheel: axis 0 0 1 -> 0 0 -1

File: ias0220_224772/urdf/differential_robot_simu_task4_part2.urdf (robot description, URDF)
Before this commit: robot IAS0220_Evgenia, 7 links, 6 joints
Joints:
- joint base_to_left_wheel: axis 0 0 1 -> 0 0 -1
