Commit message: fix typo wheels

File: ias0220_224772/urdf/differential_robot_simu_task4_part2.urdf (robot description, URDF)
Before this commit: robot IAS0220_Evgenia, 7 links, 6 joints
Joints:
- joint base_to_left_wheel: axis 0 0 -1 -> 0 0 1; child right_wheel -> left_wheel; origin xyz=0 -0.1 0 rpy=1.57 0 0 -> xyz=0 0.1 0 rpy=-1.57 0 0
- joint base_to_right_wheel: axis 0 0 1 -> 0 0 -1; child left_wheel -> right_wheel; origin xyz=0 0.1 0 rpy=-1.57 0 0 -> xyz=0 -0.1 0 rpy=1.57 0 0
