Commit message: add implementation task 8, not yet working on waypoints. odon transporf to over check

File: ias0220_224772_slam/urdf/robot.urdf (robot description, URDF)
Before this commit: robot IAS0220_Evgenia, 7 links, 6 joints
Links:
- added link sensor, mass 1e-5; collision mesh filename=package://rrbot_description/meshes/hokuyo.dae; visual mesh filename=package://rrbot_description/meshes/hokuyo.dae
Joints:
- added joint base_to_sensor: type fixed, parent base_link, child sensor, origin xyz=0 0 0.04 rpy=0 0 0
